File: robot-power-pcb-2025.kicad_sch (KiCad schematic)
At the start: 25 parts, among them J1 B14B-PHDSS, J10 B2B-PH, J11 B2B-PH, J12 B4B-PH, J13 B4B-PH, J2 XT60, J3 Conn_01x02, J4 Conn_01x02, J5 XT30, J6 XT30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

Commit message: fix schematics
Parts:
- removed K1: Relay_SPDT, symbol Relay:Relay_SPDT
- added D2: LED, LED_THT:LED_D5.0mm, symbol Device:LED
- added D3: 1N4007, Diode_THT:D_A-405_P7.62mm_Horizontal, symbol Device:D
- added J14: B2B-PH, Connector_JST:JST_PH_B2B-PH-K_1x02_P2.00mm_Vertical, symbol Connector_Generic:Conn_01x02
- added K3: SANYOU_SRD_Form_C, Relay_THT:Relay_SPDT_SANYOU_SRD_Series_Form_C, symbol Relay:SANYOU_SRD_Form_C
- added Q1: IRLZ44N, Package_TO_SOT_THT:TO-220-3_Horizontal_TabDown, symbol Transistor_FET:IRLZ44N
- added R3: 1.1k, Resistor_THT:R_Axial_DIN0207_L6.3mm_D2.5mm_P7.62mm_Horizontal, symbol Device:R
- added R4: 150R, Resistor_THT:R_Axial_DIN0207_L6.3mm_D2.5mm_P7.62mm_Horizontal, symbol Device:R
- added VR4: LM2596, Project:LM2596, symbol Project:Voltage_Regulator_Module
- C1, C2: footprint (none) -> Capacitor_THT:CP_Radial_D6.3mm_P2.50mm
- J10, J11, J7, J8, J9: footprint (none) -> Connector_JST:JST_PH_B2B-PH-K_1x02_P2.00mm_Vertical
- J12, J13: footprint (none) -> Connector_JST:JST_PH_B4B-PH-K_1x04_P2.00mm_Vertical
- J2: footprint (none) -> Connector_AMASS:AMASS_XT60-M_1x02_P7.20mm_Vertical
- J3, J4: value Conn_01x02 -> B2B-PH; footprint (none) -> Connector_JST:JST_PH_B2B-PH-K_1x02_P2.00mm_Vertical
- J5, J6: footprint (none) -> Connector_AMASS:AMASS_XT30UPB-M_1x02_P5.0mm_Vertical
- R1, R2: value R -> 10k; footprint (none) -> Resistor_THT:R_Axial_DIN0207_L6.3mm_D2.5mm_P7.62mm_Horizontal
- VR1: footprint (none) -> Project:LM2596
- VR2: footprint (none) -> Project:XHM404_Module
- VR3: value LM2596 -> XH-M404; footprint (none) -> Project:XHM404_Module
Connections:
- net GNDD is gone; now on net GND: J6.1 (Pin_1), U1.1 (~{EN}), U1.16 (GND), U2.1 (~{EN}), U2.16 (GND), U3.3 (GND), U4.3 (GND), VR1.3 (OUT-)
- net +12V: now also K3.1
- net +5V: now also U1.15 (VIO), U2.15 (VIO), Q1.3 (S), VR4.4 (OUT+); no longer J5.2 (Pin_2), VR2.4 (OUT+)
- net GND: now also D2.1 (K), D3.2 (A), K3.2, VR4.1 (IN-), VR4.3 (OUT-)
- net pump-rly: now also R4.1
- net at J3.2 (Pin_2): now also K3.4
- net at J4.2 (Pin_2): now also K3.3
- net +15V renamed +16.8V
- net +16.8V: now also J14.2 (Pin_2), R3.1, VR4.2 (IN+); no longer J2.2 (Pin_2)
- net GRB+5V: no longer names the net of U3.4 (5V)
- net GRB+5V: no longer U1.15 (VIO)
- net SC+5V: no longer names the net of U4.4 (5V)
- net SC+5V: no longer U2.15 (VIO)
- new net: J14.1 (Pin_1), J2.2 (Pin_2)
- new net: D2.2 (A), R3.2
- new net: D3.1 (K), K3.5, Q1.2 (D)
- new net: Q1.1 (G), R4.2
- new net +5VPWR: J5.2 (Pin_2), VR2.4 (OUT+)
- no-connect marks 16 -> 18
Other:
- note added: "POWER INPUT"
- note added: "POWER LED"
- note added: "PUMPS"
- moved on the sheet: C1, C2, J1, J12, J13, J3, J4, J5, J6, J7, R1, R2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

Commit message: Run to fab
Parts:
- removed D3: 1N4007, Diode_THT:D_A-405_P7.62mm_Horizontal, symbol Device:D
- removed K3: SANYOU_SRD_Form_C, Relay_THT:Relay_SPDT_SANYOU_SRD_Series_Form_C, symbol Relay:SANYOU_SRD_Form_C
- added D1: IN4007, Diode_THT:D_DO-41_SOD81_P2.54mm_Vertical_AnodeUp, symbol Device:D
- added D3, D4: IN4007, Diode_THT:D_DO-41_SOD81_P2.54mm_Vertical_AnodeUp, symbol Device:D_Small
- added H1, H2, H3, H4, H5: MountingHole, MountingHole:MountingHole_2.7mm_M2.5, symbol Mechanical:MountingHole
- added R5: 10k, Resistor_THT:R_Axial_DIN0207_L6.3mm_D2.5mm_P7.62mm_Horizontal, symbol Device:R
- J14: value B2B-PH -> XT60; footprint Connector_JST:JST_PH_B2B-PH-K_1x02_P2.00mm_Vertical -> Connector_AMASS:AMASS_XT60-M_1x02_P7.20mm_Vertical
- R4: value 150R -> 220
- U3: value Sabertooth 2X5 -> SBR-L
- U4: value Sabertooth 2X5 -> SBR-R
- VR3: value XH-M404 -> LM2596; footprint Project:XHM404_Module -> Project:LM2596
Connections:
- net +12V: now also J3.2 (Pin_2), J4.2 (Pin_2), D3.1 (K), D4.1 (K); no longer C1.1, C2.1, U1.9 (VM), U2.9 (VM)
- net +16.8V: now also C1.1, C2.1, U1.9 (VM), U2.9 (VM)
- net +5V: no longer Q1.3 (S)
- net GND: now also Q1.3 (S), D1.2 (A), R5.1; no longer J3.1 (Pin_1), J4.1 (Pin_1)
- net pump-rly: now also R5.2
- net at J8.1 (Pin_1): now also U3.9 (M1B); no longer U3.7 (M2B)
- net at J8.2 (Pin_2): now also U3.10 (M1A); no longer U3.8 (M2A)
- net at J11.1 (Pin_1): now also U4.7 (M2B); no longer U4.9 (M2B)
- net at J11.2 (Pin_2): now also U4.8 (M2A); no longer U4.10 (M2A)
- net at J9.2 (Pin_2): now also U3.8 (M2A); no longer U3.10 (M2A)
- net at J9.1 (Pin_1): now also U3.7 (M2B); no longer U3.9 (M2B)
- net at J10.1 (Pin_1): now also U4.9 (M1B); no longer U4.7 (M2B)
- net at J10.2 (Pin_2): now also U4.10 (M1A); no longer U4.8 (M2A)
- net at Q1.2 (D): now also J3.1 (Pin_1), J4.1 (Pin_1), D1.1 (K), D3.2 (A), D4.2 (A)
Other:
- moved on the sheet: J10, J11, J14, J4, J8, J9, Q1, R4

Commit message: fixes
Other:
- moved on the sheet: C1
Changed lines of the file:
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@@
 	)
 	(junction
-		(at 24.13 105.41)
+		(at 26.67 105.41)
 		(diameter 0)
 		(color 0 0 0 0)
@@
 	)
 	(junction
-		(at 24.13 97.79)
+		(at 26.67 97.79)
 		(diameter 0)
 		(color 0 0 0 0)
@@
 		)
 	)
-	(wire
-		(pts
-			(xy 20.32 97.79) (xy 24.13 97.79)
-		)
-		(stroke
-			(width 0)
-			(type default)
-		)
-	)
 	(polyline
 		(pts
@@
 		)
 	)
-	(wire
-		(pts
-			(xy 21.59 105.41) (xy 24.13 105.41)
-		)
-		(stroke
-			(width 0)
-			(type default)
-		)
-	)
 	(polyline
 		(pts
@@
 	(wire
 		(pts
-			(xy 24.13 105.41) (xy 38.1 105.41)
+			(xy 26.67 105.41) (xy 38.1 105.41)
 		)
 		(stroke
@@
 	(wire
 		(pts
-			(xy 35.56 102.87) (xy 38.1 102.87)
-		)
-		(stroke
-			(width 0)
-			(type default)
-		)
-	)
-	(wire
-		(pts
 			(xy 182.88 95.25) (xy 182.88 80.01)
 		)
@@
 	(wire
 		(pts
-			(xy 24.13 97.79) (xy 35.56 97.79)
+			(xy 26.67 97.79) (xy 38.1 97.79)
 		)
 		(stroke
@@
 	(wire
 		(pts
-			(xy 35.56 97.79) (xy 35.56 102.87)
+			(xy 38.1 97.79) (xy 38.1 102.87)
 		)
 		(stroke
@@
 		)
 	)
+	(polyline
+		(pts
+			(xy 164.084 81.28) (xy 164.084 81.534)
+		)
+		(stroke
+			(width 0)
+			(type default)
+		)
+	)
 	(wire
 		(pts
@@
 	(wire
 		(pts
+			(xy 21.59 105.41) (xy 26.67 105.41)
+		)
+		(stroke
+			(width 0)
+			(type default)
+		)
+	)
+	(wire
+		(pts
 			(xy 187.96 72.39) (xy 187.96 73.66)
 		)
@@
 		)
 	)
+	(wire
+		(pts
+			(xy 20.32 97.79) (xy 26.67 97.79)
+		)
+		(stroke
+			(width 0)
+			(type default)
+		)
+	)
 	(polyline
 		(pts
@@
 	(symbol
 		(lib_id "Device:C_Polarized")
-		(at 24.13 101.6 180)
+		(at 26.67 101.6 180)
 		(unit 1)
 		(exclude_from_sim no)
@@
 		(fields_autoplaced yes)
 		(property "Reference" "C1"
-			(at 27.94 101.2189 0)
+			(at 30.48 101.2189 0)
 			(effects
 				(font
@@
 		)
 		(property "Value" "100uF"
-			(at 27.94 103.7589 0)
+			(at 30.48 103.7589 0)
 			(effects
 				(font
@@
 		)
 		(property "Footprint" "Capacitor_THT:CP_Radial_D6.3mm_P2.50mm"
-			(at 23.1648 97.79 0)
+			(at 25.7048 97.79 0)
 			(effects
 				(font
@@
 		)
 		(property "Datasheet" "~"
-			(at 24.13 101.6 0)
+			(at 26.67 101.6 0)
 			(effects
 				(font
@@
 		)
 		(property "Description" "Polarized capacitor"
-			(at 24.13 101.6 0)
+			(at 26.67 101.6 0)
 			(effects
 				(font

Commit message: First commit
Parts:
- removed H1: MountingHole, MountingHole:MountingHole_2.7mm_M2.5, symbol Mechanical:MountingHole
- removed J1: B14B-PHDSS, Connector_JST:JST_PHD_S14B-PHDSS_2x07_P2.00mm_Horizontal, symbol Connector_Generic:Conn_02x07_Odd_Even
- removed U3: SBR-L, Project:Sabertooth_2X5, symbol Project:Sabertooth_2X5
- removed U4: SBR-R, Project:Sabertooth_2X5, symbol Project:Sabertooth_2X5
- added F1: Fuse, Fuse:Fuseholder_Cylinder-5x20mm_Schurter_0031_8201_Horizontal_Open, symbol Device:Fuse
- added PGRB1, PSC1: PH5A, Connector_JST:JST_PH_B5B-PH-K_1x05_P2.00mm_Vertical, symbol Connector_Generic:Conn_01x05
- added PMISC1: PH2A, Connector_JST:JST_PH_B2B-PH-K_1x02_P2.00mm_Vertical, symbol Connector_Generic:Conn_01x02
- added PMV1, PMV2: PH6A, Connector_JST:JST_PH_B6B-PH-K_1x06_P2.00mm_Vertical, symbol Connector_Generic:Conn_01x06
- added U3, U4: L298N_Bridge, Project:L298N_Bridge, symbol Project:L298N_Bridge
- D2: value LED -> LED_Green
- J5, J6: footprint Connector_AMASS:AMASS_XT30UPB-M_1x02_P5.0mm_Vertical -> Connector_AMASS:AMASS_XT30U-M_1x02_P5.0mm_Vertical
- R1, R2: value 10k -> 1k
- R3: value 1.1k -> 430
Connections:
- net +16.8V: now also U3.1 (+12V), U4.1 (+12V)
- net +5V: now also U3.3 (+5V), U4.3 (+5V)
- net GND: now also U3.2 (GND), U4.2 (GND); no longer U1.1 (~{EN}), U2.1 (~{EN})
- net at J14.1 (Pin_1): now also F1.1; no longer J2.2 (Pin_2)
- net at J8.1 (Pin_1): now also U3.12 (OUT3)
- net at J8.2 (Pin_2): now also U3.13 (OUT4)
- net at J11.1 (Pin_1): now also U4.12 (OUT3)
- net at J11.2 (Pin_2): now also U4.13 (OUT4)
- net at J9.1 (Pin_1): now also U3.10 (OUT1)
- net at J9.2 (Pin_2): now also U3.11 (OUT2)
- net at J10.1 (Pin_1): now also U4.10 (OUT1)
- net at J10.2 (Pin_2): now also U4.11 (OUT2)
- net grb-dir renamed GRB_DIR
- net GRB_DIR: now also PGRB1.3 (Pin_3)
- net grb-rx renamed GRB_RX
- net GRB_RX: now also PGRB1.1 (Pin_1)
- net grb-step renamed GRB_STEP
- net GRB_STEP: now also PGRB1.4 (Pin_4)
- net grb-tx renamed GRB_TX
- net GRB_TX: now also PGRB1.2 (Pin_2)
- net pump-rly renamed PUMP_RLY
- net PUMP_RLY: now also PMISC1.2 (Pin_2)
- net sc-dir renamed SC_DIR
- net SC_DIR: now also PSC1.3 (Pin_3)
- net sc-rx renamed SC_RX
- net SC_RX: now also PSC1.1 (Pin_1)
- net sc-step renamed SC_STEP
- net SC_STEP: now also PSC1.4 (Pin_4)
- net sc-tx renamed SC_TX
- net SC_TX: now also PSC1.2 (Pin_2)
- new net: F1.2, J2.2 (Pin_2)
- new net GRB_EN: PGRB1.5 (Pin_5), U1.1 (~{EN})
- new net L298N_L_ENA: PMV1.1 (Pin_1), U3.4 (ENA)
- new net L298N_L_ENB: PMV1.2 (Pin_2), U3.9 (ENB)
- new net L298N_L_IN1: PMV1.3 (Pin_3), U3.5 (IN1)
- new net L298N_L_IN2: PMV1.4 (Pin_4), U3.6 (IN2)
- new net L298N_L_IN3: PMV1.5 (Pin_5), U3.7 (IN3)
- new net L298N_L_IN4: PMV1.6 (Pin_6), U3.8 (IN4)
- new net L298N_R_ENA: PMV2.1 (Pin_1), U4.4 (ENA)
- new net L298N_R_ENB: PMV2.2 (Pin_2), U4.9 (ENB)
- new net L298N_R_IN1: PMV2.3 (Pin_3), U4.5 (IN1)
- new net L298N_R_IN2: PMV2.4 (Pin_4), U4.6 (IN2)
- new net L298N_R_IN3: PMV2.5 (Pin_5), U4.7 (IN3)
- new net L298N_R_IN4: PMV2.6 (Pin_6), U4.8 (IN4)
- new net SC_EN: PSC1.5 (Pin_5), U2.1 (~{EN})
- no-connect marks 18 -> 13
Other:
- moved on the sheet: C1, H2, H3, H4, H5, J12, J14, J8, J9, R1
