File: robot-power-pcb-2025.kicad_pcb (KiCad board)
At the start: 2 copper layers, 32 parts, among them J1 B14B-PHDSS, J10 B2B-PH, J11 B2B-PH, J12 B4B-PH, J13 B4B-PH, J14 XT60, J15 B2B-PH, J3 Conn_01x02, J4 Conn_01x02, J5 XT30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

Commit message: Run to fab
Parts:
- removed J15: B2B-PH, Connector_JST:JST_PH_B2B-PH-K_1x02_P2.00mm_Vertical
- removed K1, K3: SANYOU_SRD_Form_C, Relay_THT:Relay_SPDT_SANYOU_SRD_Series_Form_C
- removed U5, U6: L7805, Package_TO_SOT_THT:TO-220-3_Horizontal_TabUp
- added D3: IN4007, Diode_THT:D_DO-41_SOD81_P2.54mm_Vertical_AnodeUp, F.Cu at (231.0, 64.8)
- added D4: IN4007, Diode_THT:D_DO-41_SOD81_P2.54mm_Vertical_AnodeUp, F.Cu at (230.8, 55.9)
- added H1: MountingHole, MountingHole:MountingHole_2.7mm_M2.5, F.Cu at (150.0, 42.2)
- added H2: MountingHole, MountingHole:MountingHole_2.7mm_M2.5, F.Cu at (242.8, 41.8)
- added H3: MountingHole, MountingHole:MountingHole_2.7mm_M2.5, F.Cu at (150.5, 234.2)
- added H4: MountingHole, MountingHole:MountingHole_2.7mm_M2.5, F.Cu at (242.8, 234.2)
- added H5: MountingHole, MountingHole:MountingHole_2.7mm_M2.5, F.Cu at (216.2, 115.2)
- added J2: XT60, Connector_AMASS:AMASS_XT60-M_1x02_P7.20mm_Vertical, F.Cu at (240.2, 216.2)
- added Q1: IRLZ44N, Package_TO_SOT_THT:TO-220-3_Horizontal_TabDown, F.Cu at (239.8, 89.3)
- added R4: 220, Resistor_THT:R_Axial_DIN0207_L6.3mm_D2.5mm_P7.62mm_Horizontal, F.Cu at (231.8, 76.9)
- added R5: 10k, Resistor_THT:R_Axial_DIN0207_L6.3mm_D2.5mm_P7.62mm_Horizontal, F.Cu at (225.2, 84.6)
- added VR4: LM2596, Project:LM2596, F.Cu at (244.2, 124.6)
- D1: value D -> IN4007; footprint Diode_THT:D_A-405_P7.62mm_Horizontal -> Diode_THT:D_DO-41_SOD81_P2.54mm_Vertical_AnodeUp
- J3, J4: value Conn_01x02 -> B2B-PH
- U3: value Sabertooth 2X5 -> SBR-L
- U4: value Sabertooth 2X5 -> SBR-R
- moved U3 198.6 mm to (150.8, 217.9), turned to 90 degrees
- moved U4 191.0 mm to (193.1, 217.7), turned to 90 degrees
- moved VR2 171.0 mm to (221.4, 167.4), turned to 180 degrees
- moved D1 165.5 mm to (237.4, 85.8)
- moved J14 160.6 mm to (239.0, 189.8), turned to 90 degrees
- moved J7 122.6 mm to (231.5, 232.2)
- moved C1 122.3 mm to (178.3, 80.8)
- moved J10 117.1 mm to (209.0, 232.0)
- moved J11 115.5 mm to (218.2, 232.0)
- moved J4 113.2 mm to (238.4, 58.5), turned to 90 degrees
- moved D2 109.0 mm to (157.2, 43.2)
- moved C2 107.7 mm to (154.8, 81.2)
- moved R3 106.1 mm to (163.8, 39.9), turned to -90 degrees
- moved VR1 106.1 mm to (209.7, 111.7), turned to 180 degrees
- moved J3 104.1 mm to (238.5, 67.0), turned to 90 degrees
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Connections:
- C1 pad 1: +12V -> +16.8V
- C2 pad 1: +12V -> +16.8V
- J14 pad 1: GND -> Net-(J14-Pin_1)
- J14 pad 2: Net-(J14-Pin_2) -> +16.8V
- J3 pad 1: GND -> Net-(D1-K)
- J3 pad 2: Net-(J3-Pin_2) -> +12V
- J4 pad 1: GND -> Net-(D1-K)
- J4 pad 2: Net-(J4-Pin_2) -> +12V
- J5 pad 2: +5V -> +5VPWR
- J6 pad 1: GNDD -> GND
- J7 pad 2: Net-(J7-Pin_2) -> +5V
- R3 pad 1: +15V -> +16.8V
- U1 pad 1: GNDD -> GND
- U1 pad 15: GRB+5V -> +5V
- U1 pad 16: GNDD -> GND
- U1 pad 9: +12V -> +16.8V
- U2 pad 1: GNDD -> GND
- U2 pad 15: SC+5V -> +5V
- U2 pad 16: GNDD -> GND
- U2 pad 9: +12V -> +16.8V
- U3 pad 10: Net-(J9-Pin_2) -> Net-(J8-Pin_2)
- U3 pad 2: +15V -> +16.8V
- U3 pad 3: GNDD -> GND
- U3 pad 4: GRB+5V -> unconnected-(U3-5V-Pad4)
- U3 pad 7: Net-(J8-Pin_1) -> Net-(J9-Pin_1)
- U3 pad 8: Net-(J8-Pin_2) -> Net-(J9-Pin_2)
- U3 pad 9: Net-(J9-Pin_1) -> Net-(J8-Pin_1)
- U4 pad 10: Net-(J11-Pin_2) -> Net-(J10-Pin_2)
- U4 pad 2: +15V -> +16.8V
- U4 pad 3: GNDD -> GND
- U4 pad 4: SC+5V -> unconnected-(U4-5V-Pad4)
- U4 pad 7: Net-(J10-Pin_1) -> Net-(J11-Pin_1)
- U4 pad 8: Net-(J10-Pin_2) -> Net-(J11-Pin_2)
- U4 pad 9: Net-(J11-Pin_1) -> Net-(J10-Pin_1)
- VR1 pad 2: +15V -> +16.8V
- VR1 pad 3: GNDD -> GND
- VR2 pad 2: +15V -> +16.8V
- VR2 pad 4: +5V -> +5VPWR
- VR3 pad 2: +15V -> +16.8V
Routing:
- net +16.8V: track 0.00 -> 376.9 mm
- net +5V: track 0.00 -> 240.9 mm, vias 0 -> 1
- net /sbr: track 0.00 -> 126.4 mm
- net /pump-rly: track 0.00 -> 81.5 mm, vias 0 -> 1
- net Net-(D1-K): track 0.00 -> 70.2 mm
- net +12V: track 0.00 -> 64.2 mm
- net /sc-dir: track 0.00 -> 62.8 mm
- net /sc-step: track 0.00 -> 58.7 mm
- net /sc-tx: track 0.00 -> 57.1 mm
- net /sc-rx: track 0.00 -> 50.5 mm
- net /grb-dir: track 0.00 -> 48.1 mm
- net Net-(J8-Pin_2): track 0.00 -> 45.2 mm
- net /grb-step: track 0.00 -> 43.0 mm
- net Net-(J12-Pin_1): track 0.00 -> 40.3 mm
- net Net-(J8-Pin_1): track 0.00 -> 40.2 mm
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- added copper zone on B.Cu, net GND
- added copper zone on F.Cu, net GND
Other:
- board outline added: 100 x 200 mm
- board text added: "BAT"
- board text added: "BL"
- board text added: "BR"
- board text added: "ESB"
- board text added: "FL"
- board text added: "FR"
- board text added: "GRB"
- board text added: "LEDs"
- board text added: "LOGIC"
- board text added: "MOVERS"
- board text added: "POWER"
- board text added: "PUMPS"
- board text added: "SCT"
- board text added: "SERVOS"
- board text added: "STEPPERS"

Commit message: update
Other:
- board text added: "Game Team"
- board text added: "INPUT : 15-17V 20A"
- board text added: "NOTICE"
- board text added: "POWER PCB"

Commit message: fixes
Routing:
- net +16.8V: track 376.9 -> 402.0 mm, vias 0 -> 1
- net Net-(D1-K): track 70.2 -> 61.2 mm
Changed lines of the file:
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@@
 		(tags "Diode DO-41_SOD81 series Axial Vertical pin pitch 2.54mm  length 5.2mm diameter 2.7mm")
 		(property "Reference" "D1"
-			(at 1.27 -2.750635 360)
+			(at 1.27 -2.750635 0)
 			(layer "F.SilkS")
 			(effects
@@
 		)
 		(property "Value" "IN4007"
-			(at 1.27 3.639635 360)
+			(at 1.27 3.639635 0)
 			(layer "F.Fab")
 			(effects
@@
 		)
 		(fp_text user "A"
-			(at 4.64 0 360)
+			(at 4.64 0 0)
 			(layer "F.SilkS")
 			(effects
@@
 		)
 		(fp_text user "A"
-			(at 4.64 0 360)
+			(at 4.64 0 0)
 			(layer "F.Fab")
 			(effects
@@
 		)
 		(fp_text user "${REFERENCE}"
-			(at 1.27 -2.750635 360)
+			(at 1.27 -2.750635 0)
 			(layer "F.Fab")
 			(effects
@@
 		(tags "RC Connector XT30")
 		(property "Reference" "J6"
-			(at 2.5 -4 360)
+			(at 2.5 -4 0)
 			(layer "F.SilkS")
 			(effects
@@
 		)
 		(property "Value" "XT30"
-			(at 2.5 4 360)
+			(at 2.5 4 0)
 			(layer "F.Fab")
 			(effects
@@
 		)
 		(fp_text user "+"
-			(at 9 0 360)
+			(at 9 0 0)
 			(layer "F.SilkS")
 			(effects
@@
 		)
 		(fp_text user "-"
-			(at -4 0 360)
+			(at -4 0 0)
 			(layer "F.SilkS")
 			(effects
@@
 		)
 		(fp_text user "${REFERENCE}"
-			(at 2.5 0 360)
+			(at 2.5 0 0)
 			(layer "F.Fab")
 			(effects
@@
 	)
 	(gr_text "LOGIC"
-		(at 147.25 100.5 -90)
+		(at 147 102 -90)
 		(layer "F.SilkS")
 		(effects
@@
 	)
 	(segment
-		(start 237.428234 68.071766)
-		(end 237.428234 85.75)
-		(width 0.6)
-		(layer "F.Cu")
-		(net 3)
-	)
-	(segment
-		(start 238.5 67)
-		(end 237.428234 68.071766)
-		(width 0.6)
-		(layer "F.Cu")
-		(net 3)
-	)
-	(segment
 		(start 238.418234 58.468234)
 		(end 238.45 58.5)
@@
 	)
 	(segment
+		(start 238.5 67)
+		(end 237.428234 68.071766)
+		(width 0.6)
+		(layer "F.Cu")
+		(net 3)
+	)
+	(segment
 		(start 241.5 64)
 		(end 241.5 61.55)
@@
 	)
 	(segment
-		(start 231 67.29)
-		(end 237.428234 73.718234)
+		(start 237.428234 68.071766)
+		(end 237.428234 85.75)
 		(width 0.6)
 		(layer "F.Cu")
@@
 	)
 	(segment
-		(start 173.954 50.144)
-		(end 173.954 72.836)
+		(start 154.75 78.49)
+		(end 150.15 73.89)
 		(width 0.2)
 		(layer "F.Cu")
@@
 	)
 	(segment
-		(start 154.75 78.49)
-		(end 150.15 73.89)
+		(start 192.869418 82.65)
+		(end 199.1 82.65)
+		(width 0.2)
+		(layer "F.Cu")
+		(net 22)
+	)
+	(segment
+		(start 184.25 60.44)
+		(end 184.25 74.030582)
 		(width 0.2)
 		(layer "F.Cu")
@@
 	)
 	(segment
-		(start 172.35 212.9)
-		(end 172.35 210.4)
-		(width 0.6)
+		(start 163.75 39.94)
+		(end 184.25 60.44)
+		(width 0.2)
 		(layer "F.Cu")
 		(net 22)
 	)
 	(segment
-		(start 173.954 72.836)
-		(end 172.9 73.89)
-		(width 0.2)
+		(start 172.35 212.9)
+		(end 172.35 210.4)
+		(width 0.6)
 		(layer "F.Cu")
 		(net 22)
@@
 	)
 	(segment
-		(start 163.75 39.94)
-		(end 173.954 50.144)
+		(start 184.25 74.030582)
+		(end 192.869418 82.65)
 		(width 0.2)
 		(layer "F.Cu")
@@
 		(net 22)
 	)
+	(via
+		(at 180.217621 82.65)
+		(size 0.6)
+		(drill 0.3)
+		(layers "F.Cu" "B.Cu")
+		(net 22)
+	)
 	(segment
-		(start 155.85 80.15)
-		(end 154.75 81.25)
+		(start 180.217621 82.65)
+		(end 176.65 82.65)
 		(width 0.2)
 		(layer "B.Cu")
@@
 	)
 	(segment
-		(start 178.317621 80.75)
-		(end 177.717621 80.15)
+		(start 176.65 82.65)
+		(end 174.15 80.15)
+		(width 0.2)
+		(layer "B.Cu")
+		(net 22)
+	)
+	(segment
+		(start 155.85 80.15)
+		(end 154.75 81.25)
 		(width 0.2)
 		(layer "B.Cu")
@@
 	)
 	(segment
-		(start 177.717621 80.15)
+		(start 174.15 80.15)
 		(end 155.85 80.15)
 		(width 0.2)

Commit message: First commit
Parts:
- removed H1: MountingHole, MountingHole:MountingHole_2.7mm_M2.5
- removed J1: B14B-PHDSS, Connector_JST:JST_PHD_S14B-PHDSS_2x07_P2.00mm_Horizontal
- added F1: Fuse, Fuse:Fuseholder_Cylinder-5x20mm_Schurter_0031_8201_Horizontal_Open, F.Cu at (264.6, 195.4)
- added PGRB1: PH5A, Connector_JST:JST_PH_B5B-PH-K_1x05_P2.00mm_Vertical, F.Cu at (178.8, 94.4)
- added PMISC1: PH2A, Connector_JST:JST_PH_B2B-PH-K_1x02_P2.00mm_Vertical, F.Cu at (181.8, 72.3)
- added PMV1: PH6A, Connector_JST:JST_PH_B6B-PH-K_1x06_P2.00mm_Vertical, F.Cu at (177.8, 87.1)
- added PMV2: PH6A, Connector_JST:JST_PH_B6B-PH-K_1x06_P2.00mm_Vertical, F.Cu at (177.8, 79.7)
- added PSC1: PH5A, Connector_JST:JST_PH_B5B-PH-K_1x05_P2.00mm_Vertical, F.Cu at (178.8, 101.8)
- D2: value LED -> LED_Green
- J5, J6: footprint Connector_AMASS:AMASS_XT30UPB-M_1x02_P5.0mm_Vertical -> Connector_AMASS:AMASS_XT30U-M_1x02_P5.0mm_Vertical
- R1, R2: value 10k -> 1k
- R3: value 1.1k -> 430
- U3: value SBR-L -> L298N_Bridge; footprint Project:Sabertooth_2X5 -> Project:L298N_Bridge
- U4: value SBR-R -> L298N_Bridge; footprint Project:Sabertooth_2X5 -> Project:L298N_Bridge
- moved H2 213.0 mm to (175.2, 243.8)
- moved H4 184.6 mm to (267.5, 51.3)
- moved H3 117.4 mm to (267.5, 243.8)
- moved J5 115.8 mm to (266.4, 139.8)
- moved R3 97.4 mm to (258.4, 63.0), turned to 90 degrees
- moved D2 94.3 mm to (251.1, 53.2)
- moved J7 77.7 mm to (175.0, 178.8)
- moved H5 75.8 mm to (174.8, 51.8)
- moved VR2 67.4 mm to (172.7, 120.8), turned to 0 degrees
- moved U3 67.1 mm to (215.4, 236.1), turned to 0 degrees
- moved VR4 66.8 mm to (231.1, 190.2), turned to 180 degrees
- moved VR3 62.7 mm to (244.2, 126.0)
- moved J8 52.8 mm to (242.4, 241.6)
- moved U1 50.7 mm to (205.4, 78.1)
- moved U2 47.1 mm to (224.6, 78.0)
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Connections:
- net /grb-tx renamed GRB_TX
- net /pump-rly renamed PUMP_RLY
- net /sc-tx renamed SC_TX
- J2 pad 2: Net-(J14-Pin_1) -> Net-(J2-Pin_2)
- R1 pad 1: /grb-rx -> GRB_RX
- R2 pad 1: /sc-rx -> SC_RX
- U1 pad 1: GND -> GRB_EN
- U1 pad 7: /grb-step -> GRB_STEP
- U1 pad 8: /grb-dir -> GRB_DIR
- U2 pad 1: GND -> SC_EN
- U2 pad 7: /sc-step -> SC_STEP
- U2 pad 8: /sc-dir -> SC_DIR
- U3 pad 1: GND -> +16.8V
- U3 pad 10: Net-(J8-Pin_2) -> Net-(J9-Pin_1)
- U3 pad 2: +16.8V -> GND
- U3 pad 3: GND -> +5V
- U3 pad 4: unconnected-(U3-5V-Pad4) -> L298N_L_ENA
- U3 pad 5: /sbr -> L298N_L_IN1
- U3 pad 6: unconnected-(U3-S2-Pad6) -> L298N_L_IN2
- U3 pad 7: Net-(J9-Pin_1) -> L298N_L_IN3
- U3 pad 8: Net-(J9-Pin_2) -> L298N_L_IN4
- U3 pad 9: Net-(J8-Pin_1) -> L298N_L_ENB
- U4 pad 1: GND -> +16.8V
- U4 pad 10: Net-(J10-Pin_2) -> Net-(J10-Pin_1)
- U4 pad 2: +16.8V -> GND
- U4 pad 3: GND -> +5V
- U4 pad 4: unconnected-(U4-5V-Pad4) -> L298N_R_ENA
- U4 pad 5: /sbr -> L298N_R_IN1
- U4 pad 6: unconnected-(U4-S2-Pad6) -> L298N_R_IN2
- U4 pad 7: Net-(J11-Pin_1) -> L298N_R_IN3
- U4 pad 8: Net-(J11-Pin_2) -> L298N_R_IN4
- U4 pad 9: Net-(J10-Pin_1) -> L298N_R_ENB
Routing:
- net +16.8V: track 402.0 -> 0.00 mm, vias 1 -> 0
- net +5V: track 240.9 -> 72.1 mm, vias 1 -> 0
- net /sbr: track 126.4 -> 0.00 mm
- net PUMP_RLY: track 81.5 -> 0.00 mm, vias 1 -> 0
- net +12V: track 64.2 -> 0.00 mm
- net /sc-dir: track 62.8 -> 0.00 mm
- net Net-(D1-K): track 61.2 -> 0.00 mm
- net /sc-step: track 58.7 -> 0.00 mm
- net SC_TX: track 57.1 -> 0.00 mm
- net /sc-rx: track 50.5 -> 0.00 mm
- net /grb-dir: track 48.1 -> 0.00 mm
- net /grb-step: track 43.0 -> 0.00 mm
- net GRB_TX: track 34.6 -> 0.00 mm
- net /grb-rx: track 25.7 -> 0.00 mm
- net +5VPWR: track 8.30 -> 33.6 mm
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- added copper zone on B.Cu, net +16.8V
- removed copper zone on B.Cu, net GND
Other:
- board text added: "LEDS"
- board text added: "RL"
- board text added: "RR"
- board text removed: "BL"
- board text removed: "BR"
- board text removed: "FL"
- board text removed: "GRB"
- board text removed: "Game Team"
- board text removed: "INPUT : 15-17V 20A"
- board text removed: "LEDs"
- board text removed: "LOGIC"
- board text removed: "NOTICE"
- board text removed: "POWER"
- board text removed: "PUMPS"
- board text removed: "SCT"
- board text removed: "STEPPERS"

Commit message: v2
Parts:
- J7: value B2B-PH -> XT30; footprint Connector_JST:JST_PH_B2B-PH-K_1x02_P2.00mm_Vertical -> Connector_AMASS:AMASS_XT30U-M_1x02_P5.0mm_Vertical
- moved D1 20.8 mm to (249.9, 58.6), turned to 180 degrees
- moved R3 15.0 mm to (263.9, 77.0)
- moved D2 14.2 mm to (261.3, 63.0)
- moved J7 2.84 mm to (176.6, 181.2), turned to 90 degrees
- moved D4 2.23 mm to (226.0, 57.4)
- moved D3 2.20 mm to (240.1, 57.2)
- moved C1 2.07 mm to (218.2, 90.6)
- moved J3 0.15 mm to (237.8, 52.0)
Routing:
- net +5V: track 72.1 -> 277.4 mm
- net L298N_R_ENB: track 0.00 -> 188.6 mm
- net L298N_L_ENB: track 0.00 -> 184.7 mm
- net L298N_R_IN4: track 0.00 -> 176.7 mm
- net L298N_R_IN3: track 0.00 -> 174.3 mm
- net L298N_L_IN4: track 0.00 -> 173.9 mm
- net L298N_L_ENA: track 0.00 -> 173.9 mm
- net L298N_R_IN2: track 0.00 -> 172.0 mm
- net L298N_L_IN3: track 0.00 -> 171.7 mm
- net L298N_L_IN2: track 0.00 -> 171.5 mm
- net L298N_L_IN1: track 0.00 -> 171.3 mm
- net L298N_R_IN1: track 0.00 -> 169.5 mm
- net L298N_R_ENA: track 0.00 -> 165.2 mm
- net SC_TX: track 0.00 -> 80.9 mm
- net SC_DIR: track 0.00 -> 71.7 mm
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Other:
- board text added: "LOGIC PCB"
- board text added: "PCA9685"
- board text added: "PUMPS"
- board text added: "STEPPERS"
- board text removed: "POWER PCB"
- board text removed: "SERVOS"

Commit message: Add logo
Other:
- board text added: "Game Team"
- board text added: "INPUT : 14-16V ~18A"
- board text added: "In Robots, We Trust"
- board text added: "POWER PCB"
